Commit message: Add launch file for robot_state_publisher

File: ros2_ws/src/aspi_description/urdf/aspi.urdf.xacro (robot description, xacro)
@@ -61,6 +61,7 @@
             <visual>
                 <geometry>
-                    <cylinder radius="0.0275" length="0.021"/>
+                    <cylinder radius="0.0275" length="0.042"/>
                 </geometry>
+                <origin xyz="0 0 -0.0115"/>
             </visual>
         </link>
